File: Hardware/Simple faz/Simple faz.kicad_pcb (KiCad board)
At the start: 2 copper layers, 82 x 76.4 mm, 40 parts, among them J1 Entrada, J2 Re1, J3 Re1, J4 Re1, J5 Re1, K1 PR14-12V-360-1C, K2 PR14-12V-360-1C, K3 PR14-12V-360-1C, K4 PR14-12V-360-1C, Q1 MMBT2222A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

Commit message: Version Final
Parts:
- moved D4 46.5 mm to (134.3, 87.0)
- moved D6 46.5 mm to (134.6, 105.7)
- moved J1 46.5 mm to (108.1, 129.3)
- moved J4 46.5 mm to (175.6, 103.0)
- moved K3 46.5 mm to (160.0, 106.5)
- moved K4 46.5 mm to (159.9, 125.2)
- moved Q1 46.5 mm to (144.6, 73.7)
- moved Q3 46.5 mm to (144.9, 111.2)
- moved R1 46.5 mm to (144.9, 62.1)
- moved R4 46.5 mm to (144.9, 80.8)
- moved R6 46.5 mm to (135.3, 95.4)
- moved R7 46.5 mm to (144.9, 99.5)
- moved R8 46.5 mm to (139.5, 109.0)
- moved U1 46.5 mm to (142.0, 67.5)
- moved U4 46.5 mm to (142.1, 123.7)
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Routing:
- net Net-(D7-K): track 23.4 -> 27.2 mm
- net VCC: track 347.7 -> 348.4 mm
- net Net-(J5-Pin_1): track 12.0 -> 12.7 mm
- net Relay_1: track 70.2 -> 69.7 mm
- net SDA: track 32.1 -> 32.6 mm

Commit message: Ultima Versión
Parts:
- added H1: MountingHole, MountingHole:MountingHole_2.5mm, F.Cu at (98.8, 63.2)
- added H2: MountingHole, MountingHole:MountingHole_2.5mm, F.Cu at (175.9, 116.1)
- added H3: MountingHole, MountingHole:MountingHole_2.5mm, F.Cu at (98.8, 118.5)
- added H4: MountingHole, MountingHole:MountingHole_2.5mm, F.Cu at (175.4, 78.7)
- added Sensores1: Conn_01x05_Socket, Connector_PinSocket_2.54mm:PinSocket_1x05_P2.54mm_Vertical, F.Cu at (98.9, 78.8)
- U5: footprint ESP32 36PIN:MODULE_DEVKIT_V1_ESP32-WROOM-32 -> EESTN5:ESP32S
- moved SW1 10.2 mm to (125.0, 128.4), turned to 180 degrees
- moved J1 3.07 mm to (105.2, 128.1)
- moved I2C1 3.01 mm to (118.0, 68.2)
- moved R8 1.93 mm to (138.0, 110.3)
- moved R7 1.93 mm to (143.6, 101.0)
- moved U5 1.81 mm to (115.5, 96.6), turned to -90 degrees
- moved Q3 1.79 mm to (145.0, 113.0)
- moved U3 1.65 mm to (140.8, 105.7)
- moved R9 1.38 mm to (134.6, 115.0)
- moved D6 1.35 mm to (133.4, 106.4)
- moved D5 1.27 mm to (140.4, 114.0)
- moved R10 0.43 mm to (144.8, 118.7)
- moved R12 0.19 mm to (135.3, 132.8)
Connections:
- U5 pad 24: Relay_4 -> unconnected-(U5-IO2-Pad24)
- U5 pad 27: GND -> Relay_4
- U5 pad 28: unconnected-(U5-IO17-Pad28) -> Relay_3
- U5 pad 29: Relay_3 -> unconnected-(U5-IO5-Pad29)
- U5 pad 3: unconnected-(U5-SENSOR_VP-Pad3) -> Input 36
- U5 pad 4: unconnected-(U5-SENSOR_VN-Pad4) -> Input 39
- U5 pad 5: unconnected-(U5-IO34-Pad5) -> Input 34
- U5 pad 6: unconnected-(U5-IO35-Pad6) -> Input 35
- U5 pad 8: unconnected-(U5-IO33-Pad8) -> Io 33
Routing:
- net GND: track 85.5 -> 20.5 mm
- net VCC: track 348.4 -> 302.4 mm
- net Net-(J1-Pin_1): track 7.19 -> 19.8 mm
- net Relay_4: track 23.0 -> 32.6 mm
- net Io 33: track 0.00 -> 7.09 mm
- net Input 39: track 0.00 -> 5.17 mm
- net Input 36: track 0.00 -> 5.17 mm
- net Input 35: track 0.00 -> 5.17 mm
- net Input 34: track 0.00 -> 5.17 mm
- net SDA: track 32.6 -> 28.0 mm
- net Relay_1: track 69.7 -> 65.1 mm
- net SCL: track 23.1 -> 18.7 mm
- net Net-(D7-K): track 27.2 -> 23.6 mm
- net Net-(D5-K): track 23.3 -> 25.9 mm
- net Net-(D5-A): track 2.92 -> 4.75 mm
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Other:
- board size 82 x 76.4 mm -> 85 x 76.4 mm

Commit message: Version final 1.0
Parts:
- moved D5 1.11 mm to (139.2, 114.0)
- moved D8 0.97 mm to (133.4, 124.3)
- moved D4 0.92 mm to (133.4, 87.0)
- moved D1 0.88 mm to (133.4, 68.2)
- moved Q3 0.27 mm to (144.7, 113.0)
Routing:
- net VCC: track 302.4 -> 305.1 mm
- net Net-(D3-K): track 22.9 -> 24.7 mm
- net Net-(D5-A): track 4.75 -> 3.64 mm
- net Net-(D7-K): track 23.6 -> 24.7 mm
- net Net-(D1-A): track 23.7 -> 24.8 mm

Commit message: Ultima version
Routing:
- net GND: track 20.5 -> 0.00 mm
